Commit message: Update to PathOptimizer changes, correct 'with set' script

File: urdf/pr2_with_set.urdf (robot description, URDF)
Before this commit: robot pr2, 83 links, 82 joints
Links:
- added link l_marker_set; visual box size=0.026 0.026 0.026
- added link l_marker_up; visual box size=0.025 0.025 0.025
Joints:
- removed joint l_set_joint
- added joint j_marker_set: type fixed, parent l_set, child l_marker_set, origin xyz=0 0 0 rpy=0 0 0.386
- added joint j_marker_up: type fixed, parent r_gripper_r_finger_tip_link, child l_marker_up, origin xyz=0 0 0 rpy=0 0 0
- added joint j_set_joint: type fixed, parent l_gripper_palm_link, child l_set, origin xyz=0 0 0 rpy=0 -1.57079632679 -1.57079632679
