Commit message: Update documentation to gepetto-viewer-server.

File: urdf/pr2.urdf (robot description, URDF)
Before this commit: robot pr2, 82 links, 81 joints
Links:
- link bl_caster_l_wheel_link: geometry 
- link bl_caster_r_wheel_link: geometry 
- link br_caster_l_wheel_link: geometry 
- link br_caster_r_wheel_link: geometry 
- link fl_caster_l_wheel_link: geometry 
- link fl_caster_r_wheel_link: geometry 
- link fr_caster_l_wheel_link: geometry 
- link fr_caster_r_wheel_link: geometry 

Commit message: Replace PR2 continuous wrist and forearm joints by revolute

File: urdf/pr2.urdf (robot description, URDF)
Before this commit: robot pr2, 82 links, 81 joints
Joints:
- joint l_forearm_roll_joint: limit effort=30 velocity=3.6 -> lower=-3.14159265359 upper=3.14159265359 effort=30 velocity=3.6; type continuous -> revolute
- joint l_wrist_roll_joint: limit effort=10 velocity=3.6 -> lower=-3.14159 upper=3.14159 effort=10 velocity=3.6; type continuous -> revolute
- joint r_forearm_roll_joint: limit effort=30 velocity=3.6 -> lower=-3.14159 upper=3.14159 effort=30 velocity=3.6; type continuous -> revolute
- joint r_wrist_roll_joint: limit effort=10 velocity=3.6 -> lower=-3.14159265359 upper=3.14159265359 effort=10 velocity=3.6; type continuous -> revolute
